File: KiCadPrj/PowerSupplyPCB.kicad_pcb (KiCad board)
At the start: 2 copper layers, 143 x 61.9 mm, 96 parts, among them J101 Screw_Terminal_01x02, J102 Conn_02x04_Odd_Even, J201 Screw_Terminal_01x02, J301 Conn_01x05_Female, J302 Conn_01x03_Female, J303 USB_B, K201 G5Q-1, Q201 Q_NMOS_GDS, Q202 Q_NMOS_GDS, Q203 BC817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

Commit message: Changed file structure
Parts:
- added D203: D, Diode_SMD:D_SMA, F.Cu at (178.8, 58.9)
Connections:
- J201 pad 1: /Output/I_o+ -> /Output/OUT+
- J201 pad 2: /Output/OUT+ -> /Output/I_o+
- K201 pad 4: /Output/I_o+ -> (no net)
Routing:
- net /Output/OUT+: track 15.0 -> 25.7 mm
- net /Output/I_o+: track 38.8 -> 36.3 mm

Commit message: Added production files
Parts:
- moved D202 48.6 mm to (203.0, 93.3)
- moved D203 48.6 mm to (212.8, 93.7)
- moved H104 48.6 mm to (218.6, 123.3)
- moved J102 48.6 mm to (218.6, 110.6)
- moved J302 48.6 mm to (173.2, 114.9)
- moved J303 48.6 mm to (195.0, 112.8)
- moved Q201 48.6 mm to (139.8, 74.4)
- moved R205 48.6 mm to (196.8, 96.5)
- moved U304 48.6 mm to (202.1, 107.1)
- moved C203 48.6 mm to (189.3, 83.5)
- moved C314 48.6 mm to (176.9, 108.2)
- moved J201 48.6 mm to (216.8, 81.0)
- moved K201 48.6 mm to (206.9, 89.3)
- moved Q203 48.6 mm to (196.8, 93.6)
- moved R201 48.6 mm to (135.9, 74.4)
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Other:
- board text added: "Programmable Power Supply - Main Board"
- board text added: "Rev. 0.1"
- board text removed: "Programmable Power Supply - Main Board v1.0.0"
